Commit message: feat:checked movement of arm using the invuilt ik function

File: four_dof_arm.urdf (robot description, URDF)
Before this commit: robot four_dof_arm, 5 links, 4 joints
Links:
- link base_link: mass None -> 1.0
- link link1_shoulder: mass None -> 0.5
- link link2_upper_arm: mass None -> 0.75
- link link3_forearm: mass None -> 0.5
- link tool_link: mass None -> 0.1
