Commit message: feat:changes the structure and added code to get camera data

File: ik/four_dof_arm.urdf (robot description, URDF)
Before this commit: robot four_dof_arm, 5 links, 4 joints
Joints:
- removed joint joint4_wrist_roll
- added joint joint4_wrist_pitch: type revolute, parent link3_forearm, child tool_link, origin xyz=0.5 0 0 rpy=0 0 0, axis 0 1 0, limit lower=-3.14 upper=3.14 effort=50.0 velocity=1.0

Commit message: Fix.added the gripper joints and links to the arm

File: ik/four_dof_arm.urdf (robot description, URDF)
Before this commit: robot four_dof_arm, 5 links, 4 joints
Links:
- removed link tool_link
- added link gripper_base, mass 0.1; collision box size=0.04 0.08 0.02; visual box size=0.04 0.08 0.02
- added link gripper_finger_left, mass 0.05; collision box size=0.06 0.015 0.02; visual box size=0.06 0.015 0.02
- added link gripper_finger_right, mass 0.05; collision box size=0.06 0.015 0.02; visual box size=0.06 0.015 0.02
Joints:
- added joint gripper_joint_left: type prismatic, parent gripper_base, child gripper_finger_left, origin xyz=0.04 0 0 rpy=0 0 0, axis 0 1 0, limit lower=0.0 upper=0.03 effort=10.0 velocity=0.5
- added joint gripper_joint_right: type prismatic, parent gripper_base, child gripper_finger_right, origin xyz=0.04 0 0 rpy=0 0 0, axis 0 -1 0, limit lower=0.0 upper=0.03 effort=10.0 velocity=0.5
- joint joint4_wrist_pitch: child tool_link -> gripper_base

Commit message: feat:started the real model integration in sim

File: ik/four_dof_arm.urdf (robot description, URDF)
Before this commit: robot four_dof_arm_with_gripper, 7 links, 6 joints
Links:
- removed link gripper_finger_left
- removed link gripper_finger_right
- added link gripper_left; collision mesh filename=meshes/gripper_left.stl scale=0.001 0.001 0.001; visual mesh filename=meshes/gripper_left.stl scale=0.001 0.001 0.001
- added link gripper_right; collision mesh filename=meshes/gripper_right.stl scale=0.001 0.001 0.001; visual mesh filename=meshes/gripper_right.stl scale=0.001 0.001 0.001
- added link gripper_top_plate; visual mesh filename=meshes/gripper_plate_top.stl scale=0.001 0.001 0.001
- link gripper_base: mass 0.1 -> 0.05; geometry collision mesh filename=meshes/gripper_plate_bottom.stl scale=0.001 0.001 0.001; visual mesh filename=meshes/gripper_plate_bottom.stl scale=0.001 0.001 0.001
Joints:
- added joint gripper_fixed_top: type fixed, parent gripper_base, child gripper_top_plate, origin xyz=0 0 0 rpy=0 0 0
- joint gripper_joint_left: child gripper_finger_left -> gripper_left; limit lower=0.0 upper=0.03 effort=10.0 velocity=0.5 -> lower=0.0 upper=0.03 effort=20.0 velocity=0.3; origin xyz=0.04 0 0 rpy=0 0 0 -> xyz=0 0.02 0 rpy=0 0 0
- joint gripper_joint_right: child gripper_finger_right -> gripper_right; limit lower=0.0 upper=0.03 effort=10.0 velocity=0.5 -> lower=0.0 upper=0.03 effort=20.0 velocity=0.3; origin xyz=0.04 0 0 rpy=0 0 0 -> xyz=0 -0.02 0 rpy=0 0 0

Commit message: Fix.tried to make the gripper close after reaching target position instead during moving

File: ik/four_dof_arm.urdf (robot description, URDF)
Before this commit: robot four_dof_arm_with_gripper, 8 links, 7 joints
Links:
- removed link gripper_left
- removed link gripper_right
- removed link gripper_top_plate
- added link gripper_finger_left, mass 0.05; collision box size=0.06 0.015 0.02; visual box size=0.06 0.015 0.02
- added link gripper_finger_right, mass 0.05; collision box size=0.06 0.015 0.02; visual box size=0.06 0.015 0.02
- link gripper_base: mass 0.05 -> 0.1; geometry collision box size=0.04 0.08 0.02; visual box size=0.04 0.08 0.02
Joints:
- removed joint gripper_fixed_top
- joint gripper_joint_left: child gripper_left -> gripper_finger_left; limit lower=0.0 upper=0.03 effort=20.0 velocity=0.3 -> lower=0.0 upper=0.03 effort=10.0 velocity=0.5; origin xyz=0 0.02 0 rpy=0 0 0 -> xyz=0.04 0 0 rpy=0 0 0
- joint gripper_joint_right: child gripper_right -> gripper_finger_right; limit lower=0.0 upper=0.03 effort=20.0 velocity=0.3 -> lower=0.0 upper=0.03 effort=10.0 velocity=0.5; origin xyz=0 -0.02 0 rpy=0 0 0 -> xyz=0.04 0 0 rpy=0 0 0
